File: EagleFiles/MultiNavFW_9250_RevA.brd (EAGLE design)
At the start: 50.8 x 22.9 mm, 32 parts, among them IC1 24AA32ASN

Commit message: Update Eagle files
Parts:
- R3: value 10 -> 4.7k; device adafruit:R0603 -> adafruit2:R0603
- R4: value 20 -> 680; device adafruit:R0603 -> adafruit2:R0603
- R6: value 680 -> 20; device adafruit2:R0603 -> adafruit:R0603
- R7: value 4.7k -> 10; device adafruit2:R0603 -> adafruit:R0603
- moved R3 22.2 mm to (20.0, 16.2), turned to 270 degrees
- moved R7 22.2 mm to (40.6, 8.10), turned to 180 degrees
- moved R6 17.0 mm to (19.1, 6.35)
- moved R4 13.2 mm to (6.35, 4.60), turned to 270 degrees
- moved R1 13.2 mm to (6.51, 17.8), turned to 0 degrees
- moved R5 1.91 mm to (19.1, 8.26)
- renumbered IC1 to U4, U$2 to U2, U$3 to U3, USBLC6 to U1
Connections:
- net 33V: now also R3.2, R4.2; no longer R1.2, R7.2
- net GPS_BIAS: now also R7.2; no longer R3.2
- net N$1: now also R7.1; no longer R3.1
- net N$3: now also R5.1; no longer R4.1
- net N$5: now also R6.1; no longer R5.1
- net N$6: now also R1.1; no longer R6.1
- net N$9: now also R4.1; no longer R1.1
- net PPS_RAW: now also R1.2; no longer R6.2
- net SCL: now also R3.1; no longer R7.1
- net USB_DM: now also R5.2; no longer R4.2
- net USB_DP: now also R6.2; no longer R5.2
