File: EagleFiles/MultiNavFW_9250_RevA.sch (EAGLE design)
At the start: 31 parts, among them IC1 24AA32ASN

Commit message: Update Eagle files
Parts:
- R3: value 10 -> 4.7k; device adafruit:R-US_R0603 -> adafruit2:R-US_R0603
- R4: value 20 -> 680; device adafruit:R-US_R0603 -> adafruit2:R-US_R0603
- R6: value 680 -> 20; device adafruit2:R-US_R0603 -> adafruit:R-US_R0603
- R7: value 4.7k -> 10; device adafruit2:R-US_R0603 -> adafruit:R-US_R0603
- renumbered IC1 to U4, U$2 to U2, U$3 to U3, USBLC6 to U1
Connections:
- net 33V: now also R3.2, R4.2; no longer R1.2, R7.2
- net GPS_BIAS: now also R7.2; no longer R3.2
- net N$1: now also R7.1; no longer R3.1
- net N$3: now also R5.1; no longer R4.1
- net N$5: now also R6.1; no longer R5.1
- net N$6: now also R1.1; no longer R6.1
- net N$9: now also R4.1; no longer R1.1
- net PPS_RAW: now also R1.2; no longer R6.2
- net SCL: now also R3.1; no longer R7.1
- net USB_DM: now also R5.2; no longer R4.2
- net USB_DP: now also R6.2; no longer R5.2
Other:
- note added: "USBLC6"
- moved on the sheet: R1, R3, R4, R5, R6, R7
